File: zipper/hardware/v2/KiCAD/Clock Generator.sch (KiCad schematic (older format))
At the start: 32 parts, among them U1 RACON_TXCO, U12 RACON_TXCO_PLUTO+, U17 SN74LVC1G04DBVR, U18 SN74LVC1G04DBVR, U2 CDCV304PW, U3 SI5351C, U4 SN74LVC1G04DBVR, U5 SN74LVC1G04DBVR

Commit message: Updated dev kit PDF, and hardware design for placement error
Parts:
- removed R84, R86, R87, R89: 0R_0603, SM0603, symbol 0R_0603
- removed R85, R88: 0R_0603_NF, SM0603, symbol 0R_0603_NF
- added R84, R86, R87, R89: 0R_0402, R_SM0402, symbol 0R_0402
- added R85, R88: 0R_0402_NF, R_SM0402, symbol 0R_0402_NF
- C1, C2, C3, C4, C5, C6, C7, C8: footprint 0603 -> C_SM0603
- X2: renamed from U1; Component Value RACON_TXCO -> 30.72MHz_TXCO
- X3: renamed from U12; Component Value RACON_TXCO_PLUTO+ -> 30.72MHz_TXCO_P+
- renumbered U17 to U1, U18 to U12
