File: zipper/hardware/v2/KiCAD/Microcontroller.sch (KiCad schematic (older format))
At the start: 61 parts, among them J6 MINI-USB-UX60A-MB-5ST, SW2 SW, U15 AT90USB162-16AU, U16 LP5900SD-3.3, X1 8MHZ

Commit message: Updated dev kit PDF, and hardware design for placement error
Parts:
- U15: value AT90USB162-16AU -> AT90USB162-16MU; Component Value AT90USB162-16AU -> AT90USB162-16MU; Description IC, MCU, 8BIT, 16KB, FLASH, 32TQFP, -> IC, MCU, 8BIT, 16KB, FLASH, 32QFN,; Manufacturer Part Number AT90USB162-16AU -> AT90USB162-16MU; Vendor Part Number AT90USB162-16AU-ND -> AT90USB162-16MU-ND
Changed lines of the file:
@@
 Sheet 8 9
 Title "Zipper v.2"
-Date "22 oct 2013"
-Rev "0"
+Date "7 jan 2014"
+Rev "2"
 Comp ""
 Comment1 "THIS WORK IS COVERED UNDER A CREATIVE COMMONS LICENSE (CC BY 3.0)"
@@
 P 3475 4700
 F 0 "U15" H 3575 4750 60  0000 C CNN
-F 1 "AT90USB162-16AU" H 4675 5300 60  0001 C CNN
+F 1 "AT90USB162-16MU" H 4675 5300 60  0001 C CNN
 F 2 "QFN32" H 4225 4450 60  0001 C CNN
 F 3 "" H 3475 4700 60  0000 C CNN
-F 4 "IC, MCU, 8BIT, 16KB, FLASH, 32TQFP," H 4825 5050 60  0001 C CNN "Description"
-F 5 "AT90USB162-16AU" H 4725 4950 60  0001 C CNN "Manufacturer Part Number"
+F 4 "IC, MCU, 8BIT, 16KB, FLASH, 32QFN," H 4825 5050 60  0001 C CNN "Description"
+F 5 "AT90USB162-16MU" H 4725 4950 60  0001 C CNN "Manufacturer Part Number"
 F 6 "Atmel" H 4625 4850 60  0001 C CNN "Manufacturer"
 F 7 "Digi-Key" H 4475 5250 60  0001 C CNN "Vendor"
-F 8 "AT90USB162-16AU-ND" H 4675 5150 60  0001 C CNN "Vendor Part Number"
-F 9 "AT90USB162-16AU" H 4725 4750 50  0000 C CNN "Component Value"
+F 8 "AT90USB162-16MU-ND" H 4675 5150 60  0001 C CNN "Vendor Part Number"
+F 9 "AT90USB162-16MU" H 4725 4750 50  0000 C CNN "Component Value"
 	1    3475 4700
 	1    0    0    -1
