File: zipper/hardware/v2/KiCAD/Power Supply.sch (KiCad schematic (older format))
At the start: 32 parts, among them J5 JUMPER2, SW1 SW, U6 SC4524, U7 LDO1117, U8 MIC37122Y_ADJ_SOIC8

Commit message: Updated dev kit PDF, and hardware design for placement error
Parts:
- C15, C16: footprint 0805 -> C_SM0805
Changed lines of the file:
@@
 Sheet 6 9
 Title "Zipper v.2"
-Date "22 oct 2013"
-Rev "0"
+Date "7 jan 2014"
+Rev "2"
 Comp ""
 Comment1 "THIS WORK IS COVERED UNDER A CREATIVE COMMONS LICENSE (CC BY 3.0)"
@@
 F 0 "C15" H 3470 5580 50  0000 L CNN
 F 1 "1uF_C_SM0805" H 3470 5400 50  0001 L CNN
-F 2 "0805" H 3450 5500 60  0001 C CNN
+F 2 "C_SM0805" H 3450 5500 60  0001 C CNN
 F 3 "" H 3450 5500 60  0001 C CNN
 F 4 "CAP, CER, 1UF, 16V, 10%, X7R, 0805," H 3450 5500 60  0001 C CNN "Description"
@@
 F 0 "C16" H 4270 5580 50  0000 L CNN
 F 1 "1uF_C_SM0805" H 4270 5400 50  0001 L CNN
-F 2 "0805" H 4250 5500 60  0001 C CNN
+F 2 "C_SM0805" H 4250 5500 60  0001 C CNN
 F 3 "" H 4250 5500 60  0001 C CNN
 F 4 "CAP, CER, 1UF, 16V, 10%, X7R, 0805," H 4250 5500 60  0001 C CNN "Description"
